Commit message: add launch_sim

File: description/robot_core.xacro (robot description, xacro)
@@ -42,5 +42,5 @@
     </link>
     <gazebo reference="chassis">
-         <material>Gazebo/White</material>
+         <material>Gazebo/Orange</material>
     </gazebo>
     <!-- LEFT WHEEL LINK -->
@@ -112,3 +112,8 @@
         </xacro:inertial_sphere>
     </link>
+    <gazebo reference="caster_wheel">
+        <material>Gazebo/Black</material>
+        <mu1 value="0.001"/>
+        <mu2 value="0.001"/>
+    /</gazebo>
 </robot>
